Commit message: change colours

File: fishbot_description/urdf/fishbot/base.urdf.xacro (robot description, xacro)
@@ -49,4 +49,7 @@
             <child link="base_link"/>
         </joint>
+        <gazebo reference="base_link">
+            <material>Gazebo/Blue</material>
+        </gazebo>
     </xacro:macro>
 </robot>

File: fishbot_description/urdf/fishbot/sensor/laser.urdf.xacro (robot description, xacro)
@@ -85,5 +85,5 @@
         <!-- laser's colour in gazebo -->
         <gazebo reference="laser_cylinder_link">
-            <material>Gazebo/Black</material>
+            <material>Gazebo/Yellow</material>
         </gazebo>
         <gazebo reference="laser_link">
